File: misfits.kicad_pcb (KiCad board)
At the start: 4 copper layers, 40 x 30 mm, 43 parts, among them J1 GT-USB-7010B, J2 S2B-PH-K-S_LF__SN_, J3 FH34SRJ-24S-0.5SH_50_, Q1 2N7002K-7, U1 ESP32-S3-MINI-1-N8, U2 BQ24040DSQR, U3 TLV75801PDRVR, U4 ESD7104MUTAG

Commit message: Fix gnd copper fill zones and esd protection placement
ESD protection placement was wrong, and the default "remove islands"
crap from KiCAD (why the fuck is *that* the default?) failed to provide
proper ground connections. These issues have been fixed now.

Signed-off-by: Lucy <user@domain.tld>
Parts:
- U4: moved to F.Cu
- moved U4 4.69 mm to (150.2, 100.8), turned to 90 degrees
Routing:
- net /3V3: track 41.3 -> 56.7 mm
- net /USB_D_P: track 26.8 -> 24.7 mm, vias 1 -> 0
- net /USB_D_N: track 28.6 -> 26.6 mm, vias 1 -> 0
- net /5V_IN: track 18.5 -> 19.0 mm, vias 2 -> 1
