File: misfits.kicad_pcb (KiCad board)
At the start: 4 copper layers, 40 x 30 mm, 43 parts, among them J1 GT-USB-7010B, J2 S2B-PH-K-S_LF__SN_, J3 FH34SRJ-24S-0.5SH_50_, Q1 2N7002K-7, U1 ESP32-S3-MINI-1-N8, U2 BQ24040DSQR, U3 TLV75801PDRVR, U4 ESD7104MUTAG

Commit message: Move Silkscreen around, add 3d models for things that need it
Signed-off-by: Lucy Mielke <user@domain.tld>
Parts:
- moved C6 11.1 mm to (164.6, 97.6), turned to 0 degrees
Routing:
- net GND: track 0.00 -> 34.4 mm, vias 53 -> 40
- net Net-(U1-EN): track 25.4 -> 24.8 mm
