File: misfits.kicad_sch (KiCad schematic)
At the start: 43 parts, among them J1 GT-USB-7010B, J2 S2B-PH-K-S_LF__SN_, J3 FH34SRJ-24S-0.5SH_50_, Q1 2N7002K-7, U1 ESP32-S3-MINI-1-N8, U2 BQ24040DSQR, U3 TLV75801PDRVR, U4 ESD7104MUTAG

Commit message: chematics: correct R8 to 2.2 Ohms
Signed-off-by: Lucy <user@domain.tld>
Parts:
- R8: value 2.2k -> 2.2
Changed lines of the file:
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@@
 			)
 		)
-		(property "Value" "2.2k"
+		(property "Value" "2.2"
 			(at 176.53 143.5099 90)
 			(effects
