File: misfits.kicad_sch (KiCad schematic)
At the start: 43 parts, among them J1 GT-USB-7010B, J2 S2B-PH-K-S_LF__SN_, J3 FH34SRJ-24S-0.5SH_50_, Q1 2N7002K-7, U1 ESP32-S3-MINI-1-N8, U2 BQ24040DSQR, U3 TLV75801PDRVR, U4 ESD7104MUTAG

Commit message: Fix wrong resistor value, change font and orient text correctly
Signed-off-by: Lucy Mielke <user@domain.tld>
Parts:
- C11, C9: value 0.47uF -> 4.7uF
- J2: DESCRIPTION Connector Header Through Hole, Right Angle 2 position -> (none)
- R2: value 2k -> 2K; VALUE 2K -> (none)
- R6: value 200k -> 200K Ohms; VALUE 200K Ohms -> (none)
- R8: value 2.2k -> 2.2R

Commit message: Parameterize schematic/PCB layout metadata
Signed-off-by: Lucy Mielke <user@domain.tld>
Other:
- company: Red lucy -> ${AUTHOR}
- title: "Misfits" -> ${TITLE}
Changed lines of the file:
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@@
 	(paper "A4")
 	(title_block
-		(title "\"Misfits\"")
-		(date "2026-03-14")
-		(rev "2")
-		(company "Red lucy")
-		(comment 1 "redlucy404.de")
+		(title "${TITLE}")
+		(date "${CURRENT_DATE}")
+		(rev "${REVISION}")
+		(company "${AUTHOR}")
+		(comment 1 "${COMMENT1}")
 	)
 	(rectangle

Commit message: add MPN for parts that matter
Signed-off-by: Lucy Mielke <user@domain.tld>
Parts:
- J1: MP GT-USB-7010B -> (none); MPN (none) -> C963217
- J2: MP S2B-PH-K-S(LF)(SN) -> (none); MPN (none) -> C173752
- J3: MPN (none) -> C324726
- L1: MP 744043470 -> (none); MPN (none) -> C2046935
- S1, S2, S3, S4: MPN (none) -> C79150
- U1: MP ESP32-S3-MINI-1-N8 -> C2913206
- U2: MP BQ24040DSQR -> (none); MPN (none) -> C81080
- U3: MP TLV75801PDRVR -> (none); MPN (none) -> C2876308
- U4: MPN (none) -> C328026
Changed lines of the file:
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@@
 			)
 		)
-		(property "MP" "S2B-PH-K-S(LF)(SN)"
+		(property "Description_1" "Connector Header Through Hole, Right Angle 2 position"
 			(at 110.49 71.12 0)
 			(hide yes)
@@
 			)
 		)
-		(property "Description_1" "Connector Header Through Hole, Right Angle 2 position"
+		(property "Availability" "In Stock"
 			(at 110.49 71.12 0)
 			(hide yes)
@@
 			)
 		)
-		(property "Availability" "In Stock"
+		(property "AVAILABILITY" "Unavailable"
 			(at 110.49 71.12 0)
 			(hide yes)
@@
 			)
 		)
-		(property "AVAILABILITY" "Unavailable"
+		(property "MPN" "C173752"
 			(at 110.49 71.12 0)
 			(hide yes)
@@
 					(size 1.27 1.27)
 				)
-				(justify bottom)
 			)
 		)
@@
 			)
 		)
+		(property "MPN" "C79150"
+			(at 172.72 46.99 0)
+			(hide yes)
+			(show_name no)
+			(do_not_autoplace no)
+			(effects
+				(font
+					(size 1.27 1.27)
+				)
+			)
+		)
 		(pin "1_1"
 		)
@@
 			)
 		)
+		(property "MPN" "C79150"
+			(at 259.08 53.34 0)
+			(hide yes)
+			(show_name no)
+			(do_not_autoplace no)
+			(effects
+				(font
+					(size 1.27 1.27)
+				)
+			)
+		)
 		(pin "1_1"
 		)
@@
 			)
 		)
-		(property "MP" "TLV75801PDRVR"
+		(property "MPN" "C2876308"
 			(at 57.15 109.22 0)
 			(hide yes)
@@
 					(size 1.27 1.27)
 				)
-				(justify bottom)
 			)
 		)
@@
 			)
 		)
-		(property "MP" "ESP32-S3-MINI-1-N8"
+		(property "Description_1" "Bluetooth, WiFi 802.11b/g/n, Bluetooth v5.0 Transceiver Module 2.4GHz PCB Trace Surface Mount"
 			(at 228.6 55.88 0)
 			(hide yes)
@@
 			)
 		)
-		(property "Description_1" "Bluetooth, WiFi 802.11b/g/n, Bluetooth v5.0 Transceiver Module 2.4GHz PCB Trace Surface Mount"
+		(property "Availability" "In Stock"
 			(at 228.6 55.88 0)
 			(hide yes)
@@
 			)
 		)
-		(property "Availability" "In Stock"
+		(property "MANUFACTURER" "Espressif"
 			(at 228.6 55.88 0)
 			(hide yes)
@@
 			)
 		)
-		(property "MANUFACTURER" "Espressif"
+		(property "MP" "C2913206"
 			(at 228.6 55.88 0)
 			(hide yes)
@@
 					(size 1.27 1.27)
 				)
-				(justify bottom)
 			)
 		)
@@
 			)
 		)
-		(property "MP" "BQ24040DSQR"
+		(property "Availability" "In Stock"
 			(at 67.31 41.91 0)
 			(hide yes)
@@
 			)
 		)
-		(property "Availability" "In Stock"
+		(property "Check_prices" "https://www.snapeda.com/parts/BQ24040DSQR/Texas+Instruments/view-part/?ref=eda"
 			(at 67.31 41.91 0)
 			(hide yes)
@@
 			)
 		)
-		(property "Check_prices" "https://www.snapeda.com/parts/BQ24040DSQR/Texas+Instruments/view-part/?ref=eda"
+		(property "MPN" "C81080"
 			(at 67.31 41.91 0)
 			(hide yes)
@@
 					(size 1.27 1.27)
 				)
-				(justify bottom)
 			)
 		)
@@
 			)
 		)
+		(property "MPN" "C324726"
+			(at 269.24 124.46 0)
+			(hide yes)
+			(show_name no)
+			(do_not_autoplace no)
+			(effects
+				(font
+					(size 1.27 1.27)
+				)
+			)
+		)
 		(pin "21"
 		)
@@
 			)
 		)
+		(property "MPN" "C79150"
+			(at 172.72 30.48 0)
+			(hide yes)
+			(show_name no)
+			(do_not_autoplace no)
+			(effects
+				(font
+					(size 1.27 1.27)
+				)
+			)
+		)
 		(pin "1_1"
 		)
@@
 			)
 		)
+		(property "MPN" "C79150"
+			(at 259.08 48.26 0)
+			(hide yes)
+			(show_name no)
+			(do_not_autoplace no)
+			(effects
+				(font
+					(size 1.27 1.27)
+				)
+			)
+		)
 		(pin "1_1"
 		)
@@
 			)
 		)
-		(property "MP" "GT-USB-7010B"
+		(property "Description_1" "Horizontal Type-C 16P Female SMT"
 			(at 46.99 170.18 0)
 			(hide yes)
@@
 			)
 		)
-		(property "Description_1" "Horizontal Type-C 16P Female SMT"
+		(property "Availability" "Not in stock"
 			(at 46.99 170.18 0)
 			(hide yes)
@@
 			)
 		)
-		(property "Availability" "Not in stock"
+		(property "MANUFACTURER" "G-switch"
 			(at 46.99 170.18 0)
 			(hide yes)
@@
 			)
 		)
-		(property "MANUFACTURER" "G-switch"
+		(property "MPN" "C963217"
 			(at 46.99 170.18 0)
 			(hide yes)
@@
 					(size 1.27 1.27)
 				)
-				(justify bottom)
 			)
 		)
@@
 			)
 		)
-		(property "MP" "744043470"
+		(property "MPN" "C2046935"
 			(at 160.02 109.22 0)
 			(hide yes)
@@
 			)
 		)
+		(property "MPN" "C328026"
+			(at 115.57 172.72 0)
+			(hide yes)
+			(show_name no)
+			(do_not_autoplace no)
+			(effects
+				(font
+					(size 1.27 1.27)
+				)
+			)
+		)

Commit message: add MPN to PCB editor view as well for bom
Signed-off-by: Lucy Mielke <user@domain.tld>
Parts:
- D2, D3, D4: Availability In Stock -> (none); Check_prices https://www.snapeda.com/parts/B0530W-7-F/Diodes+Inc./view-p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 -> (none); Description_1 Diode Schottky 30V 0.5A 2Pin SOD123 | Diodes Inc B0530W-7-F -> (none); MANUFACTURER DIODES -> (none); MF Diodes Inc. -> (none); MP B0530W-7-F -> (none); MPN (none) -> C124188; PARTREV 9-2 -> (none); Package SOD-123 Fairchild Semiconductor -> (none); Price None -> (none); STANDARD IPC-7351B -> (none); SnapEDA_Link https://www.snapeda.com/parts/B0530W-7-F/Diodes+Inc./view-p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 -> (none)
- J1: Availability Not in stock -> (none); Check_prices https://www.snapeda.com/parts/GT-USB-7010B/G-switch/view-pa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 -> (none); Description_1 Horizontal Type-C 16P Female SMT -> (none); MANUFACTURER G-switch -> (none); MAXIMUM_PACKAGE_HEIGHT 3.16mm -> (none); MF G-switch -> (none); PARTREV A0 -> (none); Package None -> (none); Price None -> (none); STANDARD Manufacturer Recommendations -> (none); SnapEDA_Link https://www.snapeda.com/parts/GT-USB-7010B/G-switch/view-pa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 -> (none)
- J2: AVAILABILITY Unavailable -> (none); Availability In Stock -> (none); Check_prices https://www.snapeda.com/parts/S2B-PH-K-S(LF)(SN)/JST/view-p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 -> (none); Description_1 Connector Header Through Hole, Right Angle 2 position -> (none); MAXIMUM_PACKAGE_HEIGHT 4.8mm -> (none); MF JST Sales America Inc. -> (none); PACKAGE None -> (none); PRICE None -> (none); Package NON STANDARD-2 J.S.T. -> (none); Price None -> (none); SnapEDA_Link https://www.snapeda.com/parts/S2B-PH-K-S(LF)(SN)/JST/view-p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 -> (none)
- J3: Availability In Stock -> (none); Check_prices https://www.snapeda.com/parts/FH34SRJ-24S-0.5SH(50)/Hirose/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 -> (none); Description_1 24 Position FFC, FPC Connector Contacts, Top and Bottom 0.0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 -> (none); MANUFACTURER HRS -> (none); MF Hirose Electric -> (none); MP FH34SRJ-24S-0.5SH(50) -> (none); Package None -> (none); Price None -> (none); SnapEDA_Link https://www.snapeda.com/parts/FH34SRJ-24S-0.5SH(50)/Hirose/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 -> (none)
- L1: Availability In Stock -> (none); Check_prices https://www.snapeda.com/parts/744043470/W%25C3%25BCrth+Elek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 -> (none); Description_1 Inductors, Fixed, WE-TPC 4828 47uH .75A .25OHm | Wurth Elec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 -> (none); MF Würth Elektronik -> (none); Package 1919 Wurth Electronics -> (none); Price None -> (none); SnapEDA_Link https://www.snapeda.com/parts/744043470/W%25C3%25BCrth+Elek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 -> (none)
- Q1: Availability In Stock -> (none); Check_prices https://www.snapeda.com/parts/2N7002K-7/Diodes+Inc./view-pa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 -> (none); Description_1 MOSFET,N-Ch,Enhancement,60V,0.38A,SOT23 | Diodes Inc 2N7002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 -> (none); MANUFACTURER Diodes Inc. -> (none); MAXIMUM_PACKAGE_HIEGHT 1.1mm -> (none); MF Diodes Inc. -> (none); MP 2N7002K-7 -> (none); MPN (none) -> C85047; PARTREV 15-2 -> (none); Package SOT-23-3 Diodes Inc. -> (none); Price None -> (none); STANDARD IPC7351B -> (none); SnapEDA_Link https://www.snapeda.com/parts/2N7002K-7/Diodes+Inc./view-pa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 -> (none)
- S1, S2, S3, S4: Availability In Stock -> (none); Check_prices https://www.snapeda.com/parts/EVPAEDB2A/Panasonic/view-part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 -> (none); Description_1 Switch Tactile N.O. SPST Rectangular Button J-Bend 0.02A 15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 -> (none); MANUFACTURER Panasonic -> (none); MAXIMUM_PACKAGE_HEIGHT 1.45mm -> (none); MF Panasonic -> (none); MP EVPAEDB2A -> (none); Package None -> (none); Price None -> (none); STANDARD Manufacturer recommendations -> (none); SnapEDA_Link https://www.snapeda.com/parts/EVPAEDB2A/Panasonic/view-part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 -> (none)
- U1: Availability In Stock -> (none); Check_prices https://www.snapeda.com/parts/ESP32-S3-MINI-1-N8/Espressif+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 -> (none); Description_1 Bluetooth, WiFi 802.11b/g/n, Bluetooth v5.0 Transceiver Mod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 -> (none); MANUFACTURER Espressif -> (none); MAXIMUM_PACKAGE_HEIGHT 2.55mm -> (none); MF Espressif Systems -> (none); PARTREV v0.6 -> (none); Package None -> (none); Price None -> (none); STANDARD Manufacturer Recommendations -> (none); SnapEDA_Link https://www.snapeda.com/parts/ESP32-S3-MINI-1-N8/Espressif+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 -> (none)
- U2: Availability In Stock -> (none); Check_prices https://www.snapeda.com/parts/BQ24040DSQR/Texas+Instruments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 -> (none); Description_1 Standalone 1-cell 1-A linear battery charger with 4.2-V VBA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 -> (none); MF Texas Instruments -> (none); Package WSON-10 Texas Instruments -> (none); Price None -> (none); SnapEDA_Link https://www.snapeda.com/parts/BQ24040DSQR/Texas+Instruments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 -> (none)
- U3: Check_prices https://www.snapeda.com/parts/TLV75801PDRVR/Texas+Instrumen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 -> (none); Description_1 500-mA, low-IQ, high-accuracy, adjustable ultra-low-dropout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 -> (none); DigiKey_Part_Number 296-53047-1-ND -> (none); MF Texas Instruments -> (none); Package WSON-6 Texas Instruments -> (none); SnapEDA_Link https://www.snapeda.com/parts/TLV75801PDRVR/Texas+Instrumen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 -> (none)
- U4: Availability In Stock -> (none); CREATOR ASHISH -> (none); Check_prices https://www.snapeda.com/parts/ESD7104MUTAG/Onsemi/view-part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 -> (none); DUPLICATE SZESD7104MUTAG -> (none); Description_1 10V Clamp 1A (8/20µs) Ipp Tvs Diode Surface Mount 10-UDFN (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 -> (none); MANUFACTURER Onsemi -> (none); MAXIMUM_PACKAGE_HEIGHT 0.55mm -> (none); MF onsemi -> (none); MP ESD7104MUTAG -> (none); PARTREV 7 -> (none); Package UDFN-10 ON Semiconductor -> (none); Price None -> (none); STANDARD Manufacturer Recommendations -> (none); SnapEDA_Link https://www.snapeda.com/parts/ESD7104MUTAG/Onsemi/view-part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 -> (none)

Commit message: new manufacturing files
Signed-off-by: Lucy Mielke <user@domain.tld>
Parts:
- R6: value 200K Ohms -> 200K
Changed lines of the file:
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@@
 		(in_pos_files yes)
 		(dnp no)
-		(fields_autoplaced yes)
 		(property "Reference" "R6"
 			(at 93.98 123.1899 90)
@@
 			)
 		)
-		(property "Value" "200K Ohms"
-			(at 91.44 130.81 0)
-			(hide yes)
+		(property "Value" "200K"
+			(at 95.758 124.46 90)
 			(show_name no)
 			(do_not_autoplace no)
