File: misfits.kicad_sch (KiCad schematic)
At the start: 43 parts, among them J1 GT-USB-7010B, J2 S2B-PH-K-S_LF__SN_, J3 FH34SRJ-24S-0.5SH_50_, Q1 2N7002K-7, U1 ESP32-S3-MINI-1-N8, U2 BQ24040DSQR, U3 TLV75801PDRVR, U4 ESD7104MUTAG

Commit message: changes to standard symbols/footprints
Signed-off-by: Lucy Mielke <user@domain.tld>
Parts:
- removed C1, C2, C3, C8: 1uF, CL10A105KO8NNNC:CAPC1608X90N, symbol CL10A105KO8NNNC:CL10A105KO8NNNC
- removed C4, C6, C7: 0.1uF, CL10B104KA8NNNC:CAPC1608X90N, symbol CL10B104KA8NNNC:CL10B104KA8NNNC
- removed C5: 10uF, CL10A106MQ8NNNC:CAPC1608X90N, symbol CL10A106MQ8NNNC:CL10A106MQ8NNNC
- removed R1, R3, R4: 1k, RC0603JR-071KL:RESC1607X60N, symbol RC0603JR-071KL:RC0603JR-071KL
- removed R2: 2K, SMD-RES-2K-1_-1_10W_0603_:R0603, symbol SMD-RES-2K-1_-1_10W_0603_:SMD-RES-2K-1_-1_10W_0603_
- removed R5: 1M, RC0603FR-071ML:RESC1607X60N, symbol RC0603FR-071ML:RC0603FR-071ML
- removed R6: 200K, RC0603FR-07200KL:RESC1608X60N, symbol RC0603FR-07200KL:RC0603FR-07200KL
- added C1, C2, C3, C8: 1uF, Capacitor_SMD:C_0603_1608Metric, symbol Device:C
- added C4, C6, C7: 0.1uF, Capacitor_SMD:C_0603_1608Metric, symbol Device:C
- added C5: 10uF, Capacitor_SMD:C_0603_1608Metric, symbol Device:C
- added R1, R3, R4: 1k, Resistor_SMD:R_0603_1608Metric, symbol Device:R
- added R2: 2k, Resistor_SMD:R_0603_1608Metric, symbol Device:R
- added R5: 1M, Resistor_SMD:R_0603_1608Metric, symbol Device:R
- added R6: 200k, Resistor_SMD:R_0603_1608Metric, symbol Device:R
- D1: value KT-0603R -> RED; footprint KT-0603R:LED_KT-0603R -> LED_SMD:LED_0603_1608Metric
Connections:
- net 3V3: now also C4.1, C5.1, C8.1, R4.1, R5.1
- net 5V_IN: now also C1.1
- net GND: now also C1.2, C2.2, C3.2, C4.2, C5.2, C6.2, C7.2, C8.2, R1.2, R2.2, R6.2
- net at J2.1, U2.10 (OUT), U3.4 (EN)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: now also C2.1, C3.1, R3.1
- net at D1.A: now also R3.2
- net at S2.2, U1.4 (IO0): now also C7.1
- net at U3.2 (FB): now also R5.2, R6.1
- net at S1.2, U1.45 (EN): now also C6.1, R4.2
- net at U2.2 (ISET): now also R1.1
- net at U2.4 (PRETERM): now also R2.1
